File: Runtime_Tester/Runtime_Tester/Rntime_Tester.kicad_sch (KiCad schematic)
At the start: 25 parts, among them IC1 RT9193-33GB, J1 USBA_Male, SW1 Reset, SW2 Continue, U1 STM32F103C8Tx, U2 CAT24C256, Y1 Crystal

Commit message: more design
Parts:
- C10, C11, C12, C5, C6, C7, C8, C9: footprint (none) -> Capacitor_SMD:C_0603_1608Metric
- R1, R2, R4, R5, R6: footprint (none) -> Resistor_SMD:R_0603_1608Metric
- SW1, SW2: footprint (none) -> Button_Switch_THT:SW_Tactile_SPST_Angled_PTS645Vx83-2LFS
- Y1: footprint (none) -> Crystal:Crystal_SMD_SeikoEpson_MA505-2Pin_12.7x5.1mm
Connections:
- no-connect marks 36 -> 40
