File: Runtime_Tester/Runtime_Tester/Rntime_Tester.kicad_sch (KiCad schematic)
At the start: 8 parts, among them IC1 RT9193-33GB, J1 USB1061-XX-X-X_REVA, U1 STM32F103C8Tx, U2 CAT24C256

Commit message: added more components
Parts:
- added C10, C7, C8, C9: 100 nF, symbol Device:C_Small
- added C11, C12: C_Small, symbol Device:C_Small
- added C4: 1.1uF, Capacitor_SMD:C_0603_1608Metric, symbol Device:C
- added C5, C6: 10uF, symbol Device:C_Small
- added R1, R2, R6: R, symbol Device:R
- added R4, R5: 10k, symbol Device:R
- added SW1: Reset, symbol Switch:SW_Push
- added SW2: Continue, symbol Switch:SW_Push
- added Y1: Crystal, symbol Device:Crystal
- C1: renamed from 2.2uF; value C -> 2.2uF; footprint (none) -> Capacitor_SMD:C_0603_1608Metric
- C2: renamed from 2.2uf2; value C -> 2.2uF; footprint (none) -> Capacitor_SMD:C_0603_1608Metric
- C3: footprint (none) -> Capacitor_SMD:C_0603_1608Metric
- IC1: footprint SOT94P279X130-5N -> KiCad:SOT94P279X130-5N
- J1: value USB1061-XX-X-X_REVA -> USBA_Male
- R3: renamed from 100k1; value R -> 100k; footprint (none) -> Resistor_SMD:R_0603_1608Metric
- U2: footprint (none) -> 24C256:SOIC127P600X175-8N
Connections:
- net VCC is gone; now on net +3.3V: U1.24 (VDD), U1.36 (VDD), U1.48 (VDD), U1.9 (VDDA)
- net GND: now also J1.4 (GND), J1.5 (SHIELD), J1.6 (SHIELD__1), U2.4 (GND), C10.2, C4.2, C5.2, C6.2, C7.2, C8.2, C9.2, R1.1, R2.1, SW1.1, SW2.1
- net +3.3V: now reaches C2.1, IC1.5 (VOUT)
- net +3.3V: now also C10.1, C7.1, C8.1, C9.1, R4.1, R5.1
- net Oled_SDA: now reaches U2.5 (SDA)
- net Oled_SDA: now also U1.46 (PB9), R2.2
- net Oled_SCL: now reaches U2.6 (SCL)
- net Oled_SCL: now also U1.45 (PB8), R1.2
- net +3V3: now reaches U2.8 (VCC)
- net +3V3: now also C4.1
- net +5V: now reaches C1.1, IC1.1 (VIN), IC1.3 (EN), R3.1
- net +5V: now also J1.1 (VBUS)
- net Reset: now reaches U1.15 (PA5)
- net Reset: now also C5.1, R4.2, SW1.2
- net Continue: now reaches U1.16 (PA6)
- net Continue: now also C6.1, R5.2, SW2.2
- net OSC_IN: now reaches U1.5 (PD0)
- net OSC_IN: now also C11.1, R6.1, Y1.1
- net OSC_OUT: now reaches U1.6 (PD1)
- net OSC_OUT: now also C12.2, R6.2, Y1.2
- new net: C11.2, C12.1
- no-connect marks 40 -> 36
Other:
- note added: "Main Control"
- note added: "Power Circuit"
- note added: "USBA Connection"
- note added: "User Buttons"
- moved on the sheet: C1, C2, C3, IC1, J1, R3, U1, U2

Commit message: Organised the schematics
Parts:
- removed J1: USBA_Male, Usba_male:USBA_Male, symbol USB_A_Male:USB1061-XX-X-X_REVA
- added J1: USB1061-XX-X-X_REVA, USBA_Male:USBA_Male, symbol USBA_Male:USB1061-XX-X-X_REVA
- added J2: Conn_01x04_Pin, Connector_PinSocket_2.54mm:PinSocket_1x04_P2.54mm_Vertical, symbol Connector:Conn_01x04_Pin
- C10, C11, C12, C5, C6, C7, C8, C9: footprint (none) -> Capacitor_SMD:C_0603_1608Metric
- R1, R2, R4, R5, R6: footprint (none) -> Resistor_SMD:R_0603_1608Metric_Pad0.98x0.95mm_HandSolder
- SW1: footprint (none) -> Button_Switch_THT:SW_Tactile_SPST_Angled_PTS645Vx39-2LFS
- SW2: footprint (none) -> Button_Switch_THT:SW_Tactile_SPST_Angled_PTS645Vx58-2LFS
- Y1: footprint (none) -> Crystal:Crystal_SMD_SeikoEpson_MA505-2Pin_12.7x5.1mm
Connections:
- net +3.3V: now also J2.1 (Pin_1)
- net +5V: now also J1.1 (VBUS)
- net GND: now also J1.4 (GND), J1.5 (SHIELD), J1.6 (SHIELD__1), J2.2 (Pin_2)
- net Oled_SCL: now also J2.3 (Pin_3)
- net Oled_SDA: now also J2.4 (Pin_4)
- no-connect marks 36 -> 40

Commit message: added traces
Parts:
- R1, R2: value R -> 10K
- SW2: footprint Button_Switch_THT:SW_Tactile_SPST_Angled_PTS645Vx58-2LFS -> Button_Switch_THT:SW_Tactile_SPST_Angled_PTS645Vx39-2LFS
Connections:
- net Oled_SCL: no longer R1.2, U2.6 (SCL)
- net Oled_SDA: no longer R2.2, U2.5 (SDA)
- net EEPROM_SCL: now reaches U1.21 (PB10)
- net EEPROM_SCL: now also R1.2, U2.6 (SCL)
- net EEPROM_SDA: now reaches U1.22 (PB11)
- net EEPROM_SDA: now also R2.2, U2.5 (SDA)
- no-connect marks 40 -> 38
Changed lines of the file:
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@@
 	)
 	(no_connect
-		(at 226.06 90.17)
-	)
-	(no_connect
 		(at 142.24 44.45)
 	)
@@
 	)
 	(no_connect
-		(at 226.06 92.71)
-	)
-	(no_connect
 		(at 259.08 69.85)
 	)
@@
 	(wire
 		(pts
+			(xy 209.55 92.71) (xy 226.06 92.71)
+		)
+		(stroke
+			(width 0)
+			(type default)
+		)
+	)
+	(wire
+		(pts
 			(xy 218.44 87.63) (xy 226.06 87.63)
 		)
@@
 	(wire
 		(pts
+			(xy 209.55 90.17) (xy 226.06 90.17)
+		)
+		(stroke
+			(width 0)
+			(type default)
+		)
+	)
+	(wire
+		(pts
 			(xy 71.12 156.21) (xy 71.12 158.75)
 		)
@@
 		)
 	)
+	(label "EEPROM_SCL"
+		(at 209.55 90.17 0)
+		(fields_autoplaced yes)
+		(effects
+			(font
+				(size 1.27 1.27)
+			)
+			(justify left bottom)
+		)
+	)
 	(label "OSC_IN"
 		(at 262.89 128.27 0)
@@
 		)
 	)
-	(label "Oled_SDA"
+	(label "EEPROM_SDA"
 		(at 187.96 39.37 90)
 		(fields_autoplaced yes)
@@
 		)
 	)
-	(label "Oled_SDA"
+	(label "EEPROM_SDA"
 		(at 163.83 39.37 0)
 		(fields_autoplaced yes)
@@
 		)
 	)
-	(label "Oled_SCL"
+	(label "EEPROM_SDA"
+		(at 209.55 92.71 0)
+		(fields_autoplaced yes)
+		(effects
+			(font
+				(size 1.27 1.27)
+			)
+			(justify left bottom)
+		)
+	)
+	(label "EEPROM_SCL"
 		(at 163.83 41.91 0)
 		(fields_autoplaced yes)
@@
 		)
 	)
-	(label "Oled_SCL"
+	(label "EEPROM_SCL"
 		(at 181.61 39.37 90)
 		(fields_autoplaced yes)
@@
 		(dnp no)
 		(property "Reference" "R1"
-			(at 179.324 43.18 90)
+			(at 179.324 44.704 90)
 			(effects
 				(font
@@
 			)
 		)
-		(property "Value" "R"
-			(at 179.324 41.148 90)
+		(property "Value" "10K"
+			(at 179.07 41.402 90)
 			(effects
 				(font
@@
 			)
 		)
-		(property "Footprint" "Button_Switch_THT:SW_Tactile_SPST_Angled_PTS645Vx58-2LFS"
+		(property "Footprint" "Button_Switch_THT:SW_Tactile_SPST_Angled_PTS645Vx39-2LFS"
 			(at 62.23 161.29 0)
 			(effects
@@
 		(dnp no)
 		(property "Reference" "R2"
-			(at 185.674 43.18 90)
+			(at 185.166 44.704 90)
 			(effects
 				(font
@@
 			)
 		)
-		(property "Value" "R"
+		(property "Value" "10K"
 			(at 185.674 41.148 90)
 			(effects

Commit message: n
Connections:
- net +3V3 is gone; now on net +3.3V: C4.1, U2.8 (VCC)
Changed lines of the file:
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@@
 	(wire
 		(pts
-			(xy 152.4 30.48) (xy 152.4 34.29)
+			(xy 152.4 27.94) (xy 152.4 34.29)
 		)
 		(stroke
@@
 		)
 	)
+	(label "EEPROM_SDA"
+		(at 218.44 95.25 0)
+		(fields_autoplaced yes)
+		(effects
+			(font
+				(size 0.254 0.254)
+			)
+			(justify left bottom)
+		)
+	)
 	(label "EEPROM_SCL"
 		(at 181.61 39.37 90)
@@
 	)
 	(symbol
-		(lib_id "power:+3V3")
-		(at 152.4 30.48 0)
-		(unit 1)
-		(exclude_from_sim no)
-		(in_bom yes)
-		(on_board yes)
-		(dnp no)
-		(fields_autoplaced yes)
-		(property "Reference" "#PWR011"
-			(at 152.4 34.29 0)
-			(effects
-				(font
-					(size 1.27 1.27)
-				)
-				(hide yes)
-			)
-		)
-		(property "Value" "+3V3"
-			(at 152.4 25.4 0)
-			(effects
-				(font
-					(size 1.27 1.27)
-				)
-			)
-		)
-		(property "Footprint" ""
-			(at 152.4 30.48 0)
-			(effects
-				(font
-					(size 1.27 1.27)
-				)
-				(hide yes)
-			)
-		)
-		(property "Datasheet" ""
-			(at 152.4 30.48 0)
-			(effects
-				(font
-					(size 1.27 1.27)
-				)
-				(hide yes)
-			)
-		)
-		(property "Description" "Power symbol creates a global label with name \"+3V3\""
-			(at 152.4 30.48 0)
-			(effects
-				(font
-					(size 1.27 1.27)
-				)
-				(hide yes)
-			)
-		)
-		(pin "1"
-		)
-		(instances
-			(project ""
-				(path "/2e6d6ada-557b-4828-90ec-76102903f133"
-					(reference "#PWR011")
-					(unit 1)
-				)
-			)
-		)
-	)
-	(symbol
 		(lib_id "power:+5V")
 		(at 80.01 109.22 270)
@@
 					(unit 1)
 				)
+			)
+		)
+	)
+	(symbol
+		(lib_id "power:+3.3V")
+		(at 152.4 27.94 0)
+		(unit 1)
+		(exclude_from_sim no)
+		(in_bom yes)
+		(on_board yes)
+		(dnp no)
+		(fields_autoplaced yes)
+		(property "Reference" "#PWR011"
+			(at 152.4 31.75 0)
+			(effects
+				(font
+					(size 1.27 1.27)
+				)
+				(hide yes)
+			)
+		)
+		(property "Value" "+3.3V"
+			(at 152.4 22.86 0)
+			(effects
+				(font
+					(size 1.27 1.27)
+				)
+			)
+		)
+		(property "Footprint" ""
+			(at 152.4 27.94 0)
+			(effects
+				(font
+					(size 1.27 1.27)
+				)
+				(hide yes)
+			)
+		)
+		(property "Datasheet" ""
+			(at 152.4 27.94 0)
+			(effects
+				(font
+					(size 1.27 1.27)
+				)
+				(hide yes)
+			)
+		)
+		(property "Description" "Power symbol creates a global label with name \"+3.3V\""
+			(at 152.4 27.94 0)
+			(effects
+				(font
+					(size 1.27 1.27)
+				)
+				(hide yes)
+			)
+		)
+		(pin "1"
+		)
+		(instances
+			(project ""
+				(path "/2e6d6ada-557b-4828-90ec-76102903f133"
+					(reference "#PWR011")
+					(unit 1)
+				)
