File: Runtime_Tester/Runtime_Tester/Rntime_Tester.kicad_pcb (KiCad board)
At the start: 2 copper layers, 23 x 18 mm, 1 part, among them U1 STM32F103C8Tx

Commit message: added more components
Parts:
- added 100k1: R, Resistor_SMD:R_0603_1608Metric, F.Cu at (121.7, 88.8)
- added C1: 2.2uF, Capacitor_SMD:C_0603_1608Metric, F.Cu at (121.7, 85.3)
- added C2: 2.2uF, Capacitor_SMD:C_0603_1608Metric, F.Cu at (121.7, 81.5)
- added C3: 22nF, Capacitor_SMD:C_0603_1608Metric, F.Cu at (124.1, 89.5)
- added IC1: RT9193-33GB, KiCad:SOT94P279X130-5N, F.Cu at (125.4, 84.9)
- added J1: USBA_Male, Usba_male:USBA_Male, F.Cu at (115.4, 86.0)
- added U2: CAT24C256, 24C256:SOIC127P600X175-8N, F.Cu at (147.5, 99.5)
- moved U1 4.45 mm to (133.4, 85.8)
Other:
- board size 23 x 18 mm -> 2.5 x 12.4 mm

Commit message: Organised the schematics
Parts:
- removed 100k1: R, Resistor_SMD:R_0603_1608Metric
- added C10: 100 nF, Capacitor_SMD:C_0603_1608Metric, F.Cu at (93.8, 54.3)
- added C11: C_Small, Capacitor_SMD:C_0603_1608Metric, F.Cu at (93.7, 60.6)
- added C12: C_Small, Capacitor_SMD:C_0603_1608Metric, F.Cu at (95.0, 57.7)
- added C4: 1.1uF, Capacitor_SMD:C_0603_1608Metric, F.Cu at (63.4, 60.4)
- added C5: 10uF, Capacitor_SMD:C_0603_1608Metric, F.Cu at (71.5, 57.2)
- added C6: 10uF, Capacitor_SMD:C_0603_1608Metric, F.Cu at (76.5, 59.5)
- added C7: 100 nF, Capacitor_SMD:C_0603_1608Metric, F.Cu at (88.4, 62.7)
- added C8: 100 nF, Capacitor_SMD:C_0603_1608Metric, F.Cu at (79.6, 59.0)
- added C9: 100 nF, Capacitor_SMD:C_0603_1608Metric, F.Cu at (84.3, 50.4)
- added J2: Conn_01x04_Pin, Connector_PinSocket_2.54mm:PinSocket_1x04_P2.54mm_Vertical, F.Cu at (67.2, 53.8)
- added R1: R, Resistor_SMD:R_0603_1608Metric_Pad0.98x0.95mm_HandSolder, F.Cu at (61.3, 60.7)
- added R2: R, Resistor_SMD:R_0603_1608Metric_Pad0.98x0.95mm_HandSolder, F.Cu at (59.1, 60.8)
- added R3: 100k, Resistor_SMD:R_0603_1608Metric, F.Cu at (53.7, 52.6)
- added R4: 10k, Resistor_SMD:R_0603_1608Metric_Pad0.98x0.95mm_HandSolder, F.Cu at (76.6, 57.4)
- added R5: 10k, Resistor_SMD:R_0603_1608Metric_Pad0.98x0.95mm_HandSolder, F.Cu at (71.7, 59.5)
- added R6: R, Resistor_SMD:R_0603_1608Metric_Pad0.98x0.95mm_HandSolder, F.Cu at (92.7, 57.8)
- added SW1: Reset, Button_Switch_THT:SW_Tactile_SPST_Angled_PTS645Vx39-2LFS, F.Cu at (72.5, 51.4)
- added SW2: Continue, Button_Switch_THT:SW_Tactile_SPST_Angled_PTS645Vx58-2LFS, F.Cu at (76.8, 65.4)
- added Y1: Crystal, Crystal:Crystal_SMD_SeikoEpson_MA505-2Pin_12.7x5.1mm, F.Cu at (100.4, 57.2)
- J1: value USBA_Male -> USB1061-XX-X-X_REVA; footprint Usba_male:USBA_Male -> USBA_Male:USBA_Male
- moved U2 96.7 mm to (61.6, 55.1), turned to -90 degrees
- moved IC1 75.2 mm to (55.2, 58.1)
- moved C3 74.8 mm to (54.6, 61.8)
- moved J1 72.6 mm to (48.4, 57.9)
- moved C2 71.5 mm to (56.3, 52.7)
- moved C1 70.5 mm to (54.5, 63.8), turned to 0 degrees
- moved U1 55.7 mm to (86.0, 56.4), turned to 180 degrees
Connections:
- U1 pad 15: unconnected-(U1-PA5-Pad15) -> /Reset
- U1 pad 16: unconnected-(U1-PA6-Pad16) -> /Continue
- U1 pad 24: VCC -> +3.3V
- U1 pad 36: VCC -> +3.3V
- U1 pad 45: unconnected-(U1-PB8-Pad45) -> /Oled_SCL
- U1 pad 46: unconnected-(U1-PB9-Pad46) -> /Oled_SDA
- U1 pad 48: VCC -> +3.3V
- U1 pad 5: unconnected-(U1-PD0-Pad5) -> /OSC_IN
- U1 pad 6: unconnected-(U1-PD1-Pad6) -> /OSC_OUT
- U1 pad 9: VCC -> +3.3V
- U2 pad 4: unconnected-(U2-GND-Pad4) -> GND
- U2 pad 5: unconnected-(U2-SDA-Pad5) -> /Oled_SDA
- U2 pad 6: unconnected-(U2-SCL-Pad6) -> /Oled_SCL
- U2 pad 8: unconnected-(U2-VCC-Pad8) -> +3V3
Routing:
- net GND: track 0.00 -> 43.9 mm
- net /OSC_OUT: track 0.00 -> 14.9 mm
- net /OSC_IN: track 0.00 -> 14.2 mm
- net +3.3V: track 0.00 -> 13.5 mm
- net +5V: track 0.00 -> 11.5 mm
- net Net-(IC1-BP): track 0.00 -> 3.25 mm
- net Net-(C11-Pad2): track 0.00 -> 2.37 mm
- net +3V3: track 0.00 -> 1.89 mm
Other:
- board size 2.5 x 12.4 mm -> 57.2 x 19.7 mm

Commit message: added traces
Parts:
- C7, C9: value 100 nF -> 100nF
- R1, R2: value R -> 10K
- SW2: footprint Button_Switch_THT:SW_Tactile_SPST_Angled_PTS645Vx58-2LFS -> Button_Switch_THT:SW_Tactile_SPST_Angled_PTS645Vx39-2LFS
- moved R5 21.2 mm to (92.8, 61.1)
- moved C9 21.2 mm to (63.6, 54.6), turned to 90 degrees
- moved C10 19.7 mm to (75.0, 60.5)
- moved C12 19.3 mm to (76.8, 64.3)
- moved Y1 19.2 mm to (81.4, 59.9)
- moved C11 18.8 mm to (76.0, 66.9)
- moved R6 18.7 mm to (75.3, 64.5)
- moved U1 18.3 mm to (68.5, 61.8)
- moved C8 18.1 mm to (62.2, 63.9)
- moved R2 16.5 mm to (74.9, 55.9), turned to 180 degrees
- moved R4 16.3 mm to (92.8, 59.0)
- moved C7 15.9 mm to (73.1, 67.1), turned to -90 degrees
- moved C5 15.4 mm to (86.8, 59.0)
- moved SW2 15.2 mm to (91.9, 67.0)
- moved SW1 15.1 mm to (87.5, 53.0)
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Connections:
- R1 pad 2: /Oled_SCL -> /EEPROM_SCL
- R2 pad 2: /Oled_SDA -> /EEPROM_SDA
- U1 pad 21: unconnected-(U1-PB10-Pad21) -> /EEPROM_SCL
- U1 pad 22: unconnected-(U1-PB11-Pad22) -> /EEPROM_SDA
- U2 pad 5: /Oled_SDA -> /EEPROM_SDA
- U2 pad 6: /Oled_SCL -> /EEPROM_SCL
Routing:
- net +3.3V: track 13.5 -> 82.6 mm
- net /Continue: track 0.00 -> 54.1 mm
- net GND: track 43.9 -> 96.7 mm
- net /Oled_SCL: track 0.00 -> 16.4 mm
- net /Oled_SDA: track 0.17 -> 14.9 mm
- net /EEPROM_SDA: track 0.00 -> 13.9 mm
- net /Reset: track 0.00 -> 11.8 mm
- net +3V3: track 1.89 -> 11.7 mm
- net /EEPROM_SCL: track 0.00 -> 2.51 mm
- net Net-(IC1-BP): track 3.25 -> 1.85 mm
- net unconnected-(U2-WP-Pad7): track 0.00 -> 1.37 mm
- net /OSC_OUT: track 14.9 -> 15.9 mm
Other:
- board size 57.2 x 19.7 mm -> 50.3 x 19.7 mm

Commit message: pcb routing
Parts:
- removed J1: USB1061-XX-X-X_REVA, USBA_Male:USBA_Male
- added C13: 20pF, Capacitor_SMD:C_0603_1608Metric, F.Cu at (167.3, 99.9)
- added C14: 20pF, Capacitor_SMD:C_0603_1608Metric, F.Cu at (167.3, 90.7)
- added J3: 48037-2100, USBA_Male_connector:480372100, F.Cu at (117.9, 95.3)
- added Y2: Crystal, Crystal:Crystal_SMD_SeikoEpson_MA406-4Pin_11.7x4.0mm, F.Cu at (163.4, 95.3)
- C10, C8: value 100 nF -> 100nF
- C11, C12: value C_Small -> 20pF
- C4, R1, R2, U2: moved to B.Cu
- J2: value Conn_01x04_Pin -> Oled display
- R6: value R -> 1M
- Y1: footprint Crystal:Crystal_SMD_SeikoEpson_MA505-2Pin_12.7x5.1mm -> Crystal:Crystal_SMD_HC49-SD
- moved U2 102.1 mm to (161.8, 95.8), turned to 90 degrees
- moved C9 96.5 mm to (151.7, 93.8), turned to -90 degrees
- moved C8 95.4 mm to (149.9, 101.4), turned to -90 degrees
- moved C4 94.7 mm to (163.8, 90.4), turned to 90 degrees
- moved R1 94.0 mm to (161.7, 90.3), turned to -90 degrees
- moved R3 93.2 mm to (134.9, 100.3)
- moved SW1 92.2 mm to (172.2, 89.2)
- moved C6 91.8 mm to (168.8, 102.5), turned to -90 degrees
- moved SW2 91.6 mm to (176.8, 101.4)
- moved R2 91.5 mm to (159.7, 90.3), turned to -90 degrees
- moved C5 87.3 mm to (168.9, 88.6), turned to 90 degrees
- moved IC1 87.0 mm to (134.4, 95.8), turned to 90 degrees
- moved J2 86.7 mm to (138.1, 91.5)
- moved C12 85.9 mm to (154.3, 101.4)
- moved C2 85.7 mm to (133.4, 91.3)
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Connections:
- U1 pad 3: unconnected-(U1-PC14-Pad3) -> /PC14
- U1 pad 4: unconnected-(U1-PC15-Pad4) -> /PC15
Routing:
- net GND: track 96.7 -> 179.9 mm, vias 0 -> 2
- net /Reset: track 11.8 -> 48.8 mm, vias 0 -> 2
- net /PC14: track 0.00 -> 24.5 mm, vias 0 -> 2
- net /EEPROM_SCL: track 2.51 -> 26.5 mm, vias 0 -> 1
- net /PC15: track 0.00 -> 23.4 mm, vias 0 -> 2
- net /EEPROM_SDA: track 13.9 -> 26.3 mm, vias 0 -> 1
- net /Continue: track 54.1 -> 41.8 mm, vias 0 -> 2
- net +3V3: track 11.7 -> 1.95 mm
- net Net-(C13-Pad2): track 0.00 -> 8.93 mm
- net +3.3V: track 82.6 -> 75.6 mm, vias 0 -> 3
- net /OSC_IN: track 14.6 -> 21.6 mm
- net +5V: track 11.8 -> 16.8 mm
- net /Oled_SDA: track 14.9 -> 13.3 mm
- net /Oled_SCL: track 16.4 -> 15.0 mm
- net unconnected-(U2-WP-Pad7): track 1.37 -> 0.00 mm
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- added copper zone on B.Cu, net GND
- added copper zone on F.Cu, net GND
Other:
- board size 50.3 x 19.7 mm -> 56.9 x 18.4 mm
