File: Runtime_Tester/Runtime_Tester/_autosave-Rntime_Tester.kicad_pcb (KiCad board)
At the start: 2 copper layers, 50.3 x 19.7 mm, 26 parts, among them IC1 RT9193-33GB, J1 USB1061-XX-X-X_REVA, J2 Conn_01x04_Pin, SW1 Reset, SW2 Continue, U1 STM32F103C8Tx, U2 CAT24C256, Y1 Crystal

Commit message: n
Parts:
- moved SW2 19.1 mm to (91.9, 67.0), turned to 180 degrees
- moved R5 12.8 mm to (92.8, 61.1)
- moved C6 7.51 mm to (86.8, 61.3)
- moved Y1 7.44 mm to (81.4, 59.9), turned to 90 degrees
- moved C4 3.54 mm to (74.9, 57.6), turned to 180 degrees
- moved C5 3.19 mm to (86.8, 59.0), turned to 180 degrees
- moved SW1 0.97 mm to (87.5, 53.0)
- moved R2 0.56 mm to (74.9, 55.9)
- moved R1 0.54 mm to (74.8, 54.3)
Routing:
- net /Continue: track 7.19 -> 54.1 mm
- net +3.3V: track 51.7 -> 82.6 mm
- net GND: track 78.8 -> 96.7 mm
- net /Reset: track 0.34 -> 11.8 mm
- net /OSC_IN: track 25.6 -> 14.6 mm
- net +3V3: track 4.48 -> 11.7 mm
- net /OSC_OUT: track 9.81 -> 15.9 mm
- net /EEPROM_SDA: track 13.2 -> 13.9 mm
- net /EEPROM_SCL: track 1.99 -> 2.51 mm
